Commit message: Update robertbotMine_gazebo.urdf.xacro

File: robertbot_description/urdf/robertbotMine_gazebo.urdf.xacro (robot description, xacro)
@@ -0,0 +1,682 @@
+<?xml version="1.0"?>
+<robot xmlns:xacro="http://www.ros.org/wiki/xacro" name="robertbot">
+    <!--Useful Variables (Properties)-->
+    <xacro:property name="PI" value="3.14159265359" />
+    <xacro:property name="effort" value="1000" />
+    <xacro:property name="velocity" value="1" />
+    <xacro:property name="scaling" value="0.001 0.001 0.001" />
+    <xacro:macro name="default_inertial" params="mass" >
+        <inertial>
+            <mass value="${mass}" />
+            <inertia ixx="1" ixy="0" ixz="0" iyy="1" iyz="0" izz="1"/>
+        </inertial>
+    </xacro:macro>
+    <xacro:macro name="default_transmission" params="number">
+        <transmission name="transmission${number}">
+            <type>transmission_interface/SimpleTransmission</type>
+            <joint name="joint${number}">
+                <hardwareInterface>hardware_interface/PositionJointInterface</hardwareInterface>
+            </joint>
+            <actuator name="motor${number}">
+                <hardwareInterface>hardware_interface/PositionJointInterface</hardwareInterface>
+                <mechanicalReduction>1</mechanicalReduction>
+            </actuator>
+        </transmission>
+    </xacro:macro>
+    <material name="gray">
+        <color rgba="0.2 0.2 0.2 0.9" />
+    </material>
+        <material name="pinky" >
+        <color rgba="0.98 0.52 0.66 1.0" />
+    </material>
+    <material name="black" >
+        <color rgba="0.0 0.0 0.0 1.0" />
+      </material>
+    <material name="blueblue" >
+        <color rgba="0.13 0.25 0.78 1.0" />
+      </material>
+    <material name="darkgreen" >
+        <color rgba="0.019 0.28 0.02 1.0" />
+      </material>
+    <material name="coolgrey" >
+        <color rgba="0.58 0.63 0.65 1.0" />
+      </material>
+    <material name="darkgold" >
+        <color rgba="0.70 0.58 0.06 1.0" />
+    </material>
+  <material name="applegreen" >
+    <color rgba="0.4627450980392157 0.803921568627451 0.14901960784313725 1.0" />
+  </material>
+   <material name="brown" >
+     <color rgba="0.396078431372549 0.21568627450980393 0.0 1.0" />
+   </material>
+    <material name="steel">
+        <color rgba="0.75 0.75 0.75 0.30" />
+    </material>
+    <!-- Links -->
+    <link name="world" />
+        <link name="base_link_r">
+            <xacro:default_inertial mass="0.075"/>
+        <visual>
+            <origin rpy="0 4.7 0" xyz="0.045 0 0"/>
+            <geometry>
+                <mesh filename="package://robertbot_description/mesh/u_type_robot_waist_bracketr.stl" scale="${scaling}"/>
+            </geometry>
+            <material name="brown" />
+        </visual>
+        <collision>
+            <origin rpy="0 4.7 0" xyz="0.045 0 0"/>
+            <geometry>
+                <mesh filename="package://robertbot_description/mesh/u_type_robot_waist_bracketr.stl" scale="${scaling}"/>
+            </geometry>
+        </collision>
+    </link>
+    <link name="base_link_l">
+        <xacro:default_inertial mass="0.075"/>
+        <visual>
+            <origin rpy="0 -4.7 3.14" xyz="0.045 0 0"/>
+            <geometry>
+                <mesh filename="package://robertbot_description/mesh/u_type_robot_waist_bracketl.stl" scale="${scaling}"/>
+            </geometry>
+            <material name="brown" />
+        </visual>
+        <collision>
+            <origin rpy="0 -4.7 3.14" xyz="0.045 0 0"/>
+            <geometry>
+                <mesh filename="package://robertbot_description/mesh/u_type_robot_waist_bracketl.stl" scale="${scaling}"/>
+            </geometry>
+        </collision>
+    </link>
+    <link name="servo1_bracket">
+        <xacro:default_inertial mass="0.025"/>
+        <visual>
+            <origin rpy="1.57 0 0" xyz="-0.01 0.03 0"/>
+            <geometry>
+                <mesh filename="package://robertbot_description/mesh/multi_functional_servo_bracket.stl" scale="${scaling}"/>
+            </geometry>
+            <material name="coolgrey" />
+        </visual>
+        <collision>
+            <origin rpy="1.57 0 0" xyz="-0.01 0.03 0"/>
+            <geometry>
+                <mesh filename="package://robertbot_description/mesh/multi_functional_servo_bracket.stl" scale="${scaling}"/>
+            </geometry>
+            <material name="coolgrey" />
+        </collision>
+    </link>
+    <link name="servo1">
+        <xacro:default_inertial mass="0.05"/>
+        <visual>
+            <origin rpy="0 0 0" xyz="0 0 0"/>
+            <geometry>
+                <mesh filename="package://robertbot_description/mesh/mg996r_servo.stl" scale="${scaling}"/>
+            </geometry>
+            <material name="coolgrey" />
+        </visual>
+        <collision>
+            <origin rpy="0 0 0" xyz="0 0 0"/>
+            <geometry>
+                <mesh filename="package://robertbot_description/mesh/mg996r_servo.stl" scale="${scaling}"/>
+            </geometry>
+            <material name="coolgrey" />
+        </collision>
+    </link>
+    <link name="servo1_horn">
+        <xacro:default_inertial mass="0.005"/>
+        <visual>
+            <origin rpy="1.57 0 0" xyz="0 0 0"/>
+            <geometry>
+                <mesh filename="package://robertbot_description/mesh/aluminum_servo_horn.stl" scale="${scaling}"/>
+            </geometry>
+            <material name="coolgrey" />
+        </visual>
+        <collision>
+            <origin rpy="1.57 0 0" xyz="0 0 0"/>
+            <geometry>
+                <mesh filename="package://robertbot_description/mesh/aluminum_servo_horn.stl" scale="${scaling}"/>
+            </geometry>
+            <material name="coolgrey" />
+        </collision>
+    </link>
+    <link name="servo2_bracket">
+        <xacro:default_inertial mass="0.025"/>
+        <visual>
+            <origin rpy="1.57 1.57 3.14" xyz="0.023 -0.04 0.024"/>
+            <geometry>
+                <mesh filename="package://robertbot_description/mesh/multi_functional_servo_bracket.stl" scale="${scaling}"/>
+            </geometry>
+            <material name="coolgrey" />
+        </visual>
+        <collision>
+            <origin rpy="1.57 1.57 3.14" xyz="0.023 -0.04 0.024"/>
+            <geometry>
+                <mesh filename="package://robertbot_description/mesh/multi_functional_servo_bracket.stl" scale="${scaling}"/>
+            </geometry>
+            <material name="coolgrey" />
+        </collision>
+    </link>
+    <link name="doublelongu_servobracketl">
+        <xacro:default_inertial mass="0.025"/>
+        <visual>
+            <origin rpy="3.14 0 0" xyz="-0.028 0.052 0.015"/>
+            <geometry>
+                <mesh filename="package://robertbot_description/mesh/long_u_type_servo_bracket.stl" scale="${scaling}"/>
+            </geometry>
+            <material name="coolgrey" />
+        </visual>
+        <collision>
+            <origin rpy="3.14 0 0" xyz="-0.028 0.052 0.015"/>
+            <geometry>
+                <mesh filename="package://robertbot_description/mesh/long_u_type_servo_bracket.stl" scale="${scaling}"/>
+            </geometry>
+            <material name="coolgrey" />
+        </collision>
+    </link>
+    <link name="doublelongu_servobracketr">
+        <xacro:default_inertial mass="0.025"/>
+        <visual>
+            <origin rpy="0 0 0" xyz="-0.028 -0.002 -0.01"/>
+            <geometry>
+                <mesh filename="package://robertbot_description/mesh/long_u_type_servo_bracket.stl" scale="${scaling}"/>
+            </geometry>
+            <material name="coolgrey" />
+        </visual>
+        <collision>
+            <origin rpy="0 0 0" xyz="-0.028 -0.002 -0.01"/>
+            <geometry>
+                <mesh filename="package://robertbot_description/mesh/long_u_type_servo_bracket.stl" scale="${scaling}"/>
+            </geometry>
+            <material name="coolgrey" />
+        </collision>
+    </link>
+    <link name="servo2">
+        <xacro:default_inertial mass="0.05"/>
+        <visual>
+            <origin rpy="0 -1.57 0" xyz="0.017 0.001 0.006"/>
+            <geometry>
+                <mesh filename="package://robertbot_description/mesh/mg996r_servo.stl" scale="${scaling}"/>
+            </geometry>
+            <material name="coolgrey" />
+        </visual>
+        <collision>
+            <origin rpy="0 -1.57 0" xyz="0.017 0.001 0.006"/>
+            <geometry>
+                <mesh filename="package://robertbot_description/mesh/mg996r_servo.stl" scale="${scaling}"/>
+            </geometry>
+            <material name="coolgrey" />
+        </collision>
+    </link>
+    <link name="servo2_horn">
+        <xacro:default_inertial mass="0.005"/>
+        <visual>
+            <origin rpy="1.57 1.57 3.14" xyz="-0.001 0.012 -0.002"/>
+            <geometry>
+                <mesh filename="package://robertbot_description/mesh/aluminum_servo_horn.stl" scale="${scaling}"/>
+            </geometry>
+            <material name="coolgrey" />
+        </visual>
+        <collision>
+            <origin rpy="1.57 1.57 3.14" xyz="-0.001 0.012 -0.002"/>
+            <geometry>
+                <mesh filename="package://robertbot_description/mesh/aluminum_servo_horn.stl" scale="${scaling}"/>
+            </geometry>
+            <material name="coolgrey" />
+        </collision>
+    </link>
+    <link name="core_u">
+        <xacro:default_inertial mass="0.23"/>
+        <visual name='ul'>
+            <origin rpy="0 1.57 1.57" xyz="0.001 -0.037 0.014"/>
+            <geometry>
+                <mesh filename="package://robertbot_description/mesh/multi_functional_servo_bracket.stl" scale="${scaling}"/>
+            </geometry>
+            <material name="coolgrey" />
+        </visual>
+        <collision name='ul'>
+            <origin rpy="0 1.57 1.57" xyz="0.001 -0.037 0.014"/>
+            <geometry>
+                <mesh filename="package://robertbot_description/mesh/multi_functional_servo_bracket.stl" scale="${scaling}"/>
+            </geometry>
+            <material name="coolgrey" />
+        </collision>
+        <visual name='core'>
+            <origin rpy="0 0 1.57" xyz="-0.0135 0.028 -0.381"/>
+            <geometry>
+                <mesh filename="package://robertbot_description/mesh/Disk_Manipulator_6DOF.stl" scale="${scaling}"/>
+            </geometry>
+            <material name="coolgrey" />
+        </visual>
+        <collision name='core'>
+            <origin rpy="0 0 1.57" xyz="-0.0135 0.028 -0.381"/>
+            <geometry>
+                <mesh filename="package://robertbot_description/mesh/Disk_Manipulator_6DOF.stl" scale="${scaling}"/>
+            </geometry>
+            <material name="coolgrey" />
+        </collision>
+        <visual name='ur'>
+            <origin rpy="0 1.57 1.57" xyz="0.0012 0.089 0.014"/>
+            <geometry>
+                <mesh filename="package://robertbot_description/mesh/multi_functional_servo_bracket.stl" scale="${scaling}"/>
+            </geometry>
+            <material name="coolgrey" />
+        </visual>
+        <collision name='ur'>
+            <origin rpy="0 1.57 1.57" xyz="0.0012 0.089 0.014"/>
+            <geometry>
+                <mesh filename="package://robertbot_description/mesh/multi_functional_servo_bracket.stl" scale="${scaling}"/>
+            </geometry>
+            <material name="coolgrey" />
+        </collision>
+        <visual name='ul_outer'>
+            <origin rpy="0 1.57 -3.14" xyz="-0.011 0.028 -0.013"/>
+            <geometry>
+                <mesh filename="package://robertbot_description/mesh/l_type_servo_bracket.stl" scale="${scaling}"/>
+            </geometry>
+            <material name="coolgrey" />
+        </visual>
+        <collision name='ul_outer'>
+            <origin rpy="0 1.57 -3.14" xyz="-0.011 0.028 -0.013"/>
+            <geometry>
+                <mesh filename="package://robertbot_description/mesh/l_type_servo_bracket.stl" scale="${scaling}"/>
+            </geometry>
+            <material name="coolgrey" />
+        </collision>
+        <visual name='ur_outer'>
+            <origin rpy="0 1.57 0" xyz="-0.036 0.081 -0.013"/>
+            <geometry>
+                <mesh filename="package://robertbot_description/mesh/l_type_servo_bracket.stl" scale="${scaling}"/>
+            </geometry>
+            <material name="coolgrey" />
+        </visual>
+        <collision name='ur_outer'>
+            <origin rpy="0 1.57 0" xyz="-0.036 0.081 -0.013"/>
+            <geometry>
+                <mesh filename="package://robertbot_description/mesh/l_type_servo_bracket.stl" scale="${scaling}"/>
+            </geometry>
+            <material name="coolgrey" />
+        </collision>
+    </link>
+    <link name="servo3">
+        <xacro:default_inertial mass="0.05"/>
+        <visual>
+            <origin rpy="0 -1.57 0" xyz="0.019 0.004 0.002"/>
+            <geometry>
+                <mesh filename="package://robertbot_description/mesh/mg996r_servo.stl" scale="${scaling}"/>
+            </geometry>
+            <material name="coolgrey" />
+        </visual>
+        <collision>
+            <origin rpy="0 -1.57 0" xyz="0.019 0.004 0.002"/>
+            <geometry>
+                <mesh filename="package://robertbot_description/mesh/mg996r_servo.stl" scale="${scaling}"/>
+            </geometry>
+            <material name="coolgrey" />
+        </collision>
+    </link>
+    <link name="servo3_horn">
+        <xacro:default_inertial mass="0.005"/>
+        <visual>
+            <origin rpy="1.57 1.57 3.14" xyz="0.001 0.015 -0.006"/>
+            <geometry>
+                <mesh filename="package://robertbot_description/mesh/aluminum_servo_horn.stl" scale="${scaling}"/>
+            </geometry>
+            <material name="coolgrey" />
+        </visual>
+        <collision>
+            <origin rpy="1.57 1.57 3.14" xyz="0.001 0.015 -0.006"/>
+            <geometry>
+                <mesh filename="package://robertbot_description/mesh/aluminum_servo_horn.stl" scale="${scaling}"/>
+            </geometry>
+            <material name="coolgrey" />
+        </collision>
+    </link>
+    <link name='bracketu4'>
+        <xacro:default_inertial mass="0.025"/>
+        <visual>
+            <origin rpy="0 0 4.7" xyz="-0.052 0.055 -0.382"/>
+            <geometry>
+                <mesh filename="package://robertbot_description/mesh/Disk_Manipulator_6DOF2.stl" scale="${scaling}"/>
+            </geometry>
+            <material name="darkgold"/>
+        </visual>
+        <collision>
+            <origin rpy="0 0 4.7" xyz="-0.052 0.055 -0.382"/>
+            <geometry>
+                <mesh filename="package://robertbot_description/mesh/Disk_Manipulator_6DOF2.stl" scale="${scaling}"/>
+            </geometry>
+            <material name="darkgold"/>
+        </collision>
+    </link>
+    <link name="servo4">
+        <xacro:default_inertial mass="0.05"/>
+        <visual>
+            <origin rpy="0 -1.57 0" xyz="0.021 -0.001 0"/>
+            <geometry>
+                <mesh filename="package://robertbot_description/mesh/mg996r_servo.stl" scale="${scaling}"/>
+            </geometry>
+            <material name="coolgrey" />
+        </visual>
+        <collision>
+            <origin rpy="0 -1.57 0" xyz="0.021 -0.001 0"/>
+            <geometry>
+                <mesh filename="package://robertbot_description/mesh/mg996r_servo.stl" scale="${scaling}"/>
+            </geometry>
+            <material name="coolgrey" />
+        </collision>
+    </link>
+    <link name="servo4_horn">
+        <xacro:default_inertial mass="0.005"/>
+        <visual>
+            <origin rpy="1.57 1.57 3.14" xyz="0.004 -0.004 0"/>
+            <geometry>
+                <mesh filename="package://robertbot_description/mesh/aluminum_servo_horn.stl" scale="${scaling}"/>
+            </geometry>
+            <material name="coolgrey" />
+        </visual>
+        <collision>
+            <origin rpy="1.57 1.57 3.14" xyz="0.004 -0.004 0"/>
+            <geometry>
+                <mesh filename="package://robertbot_description/mesh/aluminum_servo_horn.stl" scale="${scaling}"/>
+            </geometry>
+            <material name="coolgrey" />
+        </collision>
+    </link>
+    <link name="servo5">
+        <xacro:default_inertial mass="0.05"/>
+        <visual>
+            <origin rpy="-1.57 1.57 0" xyz="0 -0.027 0"/>
+            <geometry>
+                <mesh filename="package://robertbot_description/mesh/mg996r_servo.stl" scale="${scaling}"/>
+            </geometry>
+            <material name="coolgrey" />
+        </visual>
+        <collision>
+            <origin rpy="-1.57 1.57 0" xyz="0 -0.027 0"/>
+            <geometry>
+                <mesh filename="package://robertbot_description/mesh/mg996r_servo.stl" scale="${scaling}"/>
+            </geometry>
+            <material name="coolgrey" />
+        </collision>
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