Commit message: Update robertbot_gazebo.urdf.xacro

File: robertbot_description/urdf/robertbot_gazebo.urdf.xacro (robot description, xacro)
@@ -0,0 +1,964 @@
+<?xml version="1.0"?>
+<robot xmlns:xacro="http://www.ros.org/wiki/xacro" name="robertbot">
+    <!--Useful Variables (Properties)-->
+    <xacro:property name="PI" value="3.14159265359" />
+    <xacro:property name="effort" value="1000" />
+    <xacro:property name="velocity" value="1" />
+    <xacro:property name="scaling" value="0.001 0.001 0.001" />
+    <xacro:macro name="default_inertial" params="mass" >
+        <inertial>
+            <mass value="${mass}" />
+            <inertia ixx="1" ixy="0" ixz="0" iyy="1" iyz="0" izz="1"/>
+        </inertial>
+    </xacro:macro>
+    <xacro:macro name="default_transmission" params="number">
+        <transmission name="transmission_${number}">
+            <type>transmission_interface/SimpleTransmission</type>
+            <joint name="joint${number}">
+                <hardwareInterface>hardware_interface/PositionJointInterface</hardwareInterface>
+            </joint>
+            <actuator name="motor_${number}">
+                <hardwareInterface>hardware_interface/PositionJointInterface</hardwareInterface>
+                <mechanicalReduction>1</mechanicalReduction>
+            </actuator>
+        </transmission>
+    </xacro:macro>
+    <material name="gray">
+        <color rgba="0.2 0.2 0.2 0.9" />
+    </material>
+    <material name="bronze">
+        <color rgba="0.6588235294117647 0.4745098039215686 0.0 1.0" />
+    </material>
+        <material name="pinky" >
+        <color rgba="0.98 0.52 0.66 1.0" />
+    </material>
+    <material name="black" >
+        <color rgba="0.0 0.0 0.0 1.0" />
+      </material>
+    <material name="blueblue" >
+        <color rgba="0.13 0.25 0.78 1.0" />
+      </material>
+    <material name="darkgreen" >
+        <color rgba="0.019 0.28 0.02 1.0" />
+      </material>
+    <material name="coolgrey" >
+        <color rgba="0.58 0.63 0.65 1.0" />
+      </material>
+    <material name="darkgold" >
+        <color rgba="0.70 0.58 0.06 1.0" />
+    </material>
+  <material name="applegreen" >
+    <color rgba="0.4627450980392157 0.803921568627451 0.14901960784313725 1.0" />
+  </material>
+   <material name="brown" >
+     <color rgba="0.396078431372549 0.21568627450980393 0.0 1.0" />
+   </material>
+    <material name="steel">
+        <color rgba="0.75 0.75 0.75 0.30" />
+    </material>
+    <!-- Links -->
+    <link name="world"/>
+    <link name="base_link">
+        <xacro:default_inertial mass="1.0"/>
+        <visual>
+            <geometry>
+                <box size="0.33 0.23 0.15" />
+            </geometry>
+            <material name="black" />
+            <origin rpy="0 0 0" xyz="0 0 -0.075" />
+        </visual>
+        <collision>
+            <geometry>
+                <box size="0.33 0.23 0.15" />
+            </geometry>
+            <material name="black" />
+            <origin rpy="0 0 0" xyz="0 0 -0.075" />
+        </collision>
+    </link>
+    <link name="vertical_link">
+        <xacro:default_inertial mass="0.5"/>
+        <visual>
+            <geometry>
+                <box size="0.02 0.02 1.025" />
+            </geometry>
+            <material name="bronze" />
+            <origin rpy="0 0 0" xyz="0 0 0" />
+        </visual>
+        <collision>
+            <geometry>
+                <box size="0.02 0.02 1.025" />
+            </geometry>
+            <material name="bronze" />
+            <origin rpy="0 0 0" xyz="0 0 0" />
+        </collision>
+    </link>
+    <link name="beam_link">
+        <xacro:default_inertial mass="0.2"/>
+        <visual>
+            <geometry>
+                <box size="0.02 0.07 0.025" />
+            </geometry>
+            <material name="brown" />
+            <origin rpy="0 0 0" xyz="0 0 0" />
+        </visual>
+        <collision>
+            <geometry>
+                <box size="0.02 0.07 0.025" />
+            </geometry>
+            <material name="brown" />
+            <origin rpy="0 0 0" xyz="0 0 0" />
+        </collision>
+    </link>
+    <link name="rod_link">
+        <xacro:default_inertial mass="0.3"/>
+        <visual>
+            <geometry>
+                <cylinder length="0.825" radius=".004" />
+            </geometry>
+            <material name="steel" />
+            <origin rpy="0 0 0" xyz="0 0 0" />
+        </visual>
+        <collision>
+            <geometry>
+                <cylinder length="0.825" radius=".004" />
+            </geometry>
+            <material name="steel" />
+            <origin rpy="0 0 0" xyz="0 0 0" />
+        </collision>
+    </link>
+    <link name="torso_link">
+        <xacro:default_inertial mass="0.6"/>
+        <visual>
+            <geometry>
+                <box size="0.15 0.145 0.005" />
+            </geometry>
+            <material name="coolgrey" />
+            <origin rpy="0 0 0" xyz="0 0 0.055" />
+        </visual>
+        <collision>
+            <geometry>
+                <box size="0.15 0.145 0.005" />
+            </geometry>
+            <material name="coolgrey" />
+            <origin rpy="0 0 0" xyz="0 0 0.055" />
+        </collision>
+    </link>
+    <link name="camera_link">
+        <xacro:default_inertial mass="0.1"/>
+        <visual>
+            <geometry>
+                  <box size="0.06 0.28 0.035" />
+            </geometry>
+            <material name="applegreen" />
+            <origin rpy="0 0 0" xyz="0.00 -0.055 0" />
+        </visual>
+        <collision>
+            <geometry>
+                  <box size="0.06 0.28 0.035" />
+            </geometry>
+            <material name="applegreen" />
+            <origin rpy="0 0 0" xyz="0.00 -0.055 0" />
+        </collision>
+    </link>
+    <link name="wheel1">
+        <xacro:default_inertial mass="1.0"/>
+        <visual>
+            <geometry>
+                <cylinder length="0.037" radius=".04" />
+            </geometry>
+            <material name="gray" />
+            <origin rpy="1.5708 0 0" xyz="0 0 0" />
+        </visual>
+        <collision>
+            <geometry>
+                <cylinder length="0.037" radius=".04" />
+            </geometry>
+            <material name="gray" />
+            <origin rpy="1.5708 0 0" xyz="0 0 0" />
+        </collision>
+    </link>
+    <link name="wheel2">
+        <xacro:default_inertial mass="1.0"/>
+        <visual>
+            <geometry>
+                <cylinder length="0.037" radius=".04" />
+            </geometry>
+            <material name="gray" />
+            <origin rpy="1.5708 0 0" xyz="0 0 0" />
+        </visual>
+        <collision>
+            <geometry>
+                <cylinder length="0.037" radius=".04" />
+            </geometry>
+            <material name="gray" />
+            <origin rpy="1.5708 0 0" xyz="0 0 0" />
+        </collision>
+    </link>
+     <link name="wheel3">
+        <xacro:default_inertial mass="1.0"/>
+        <visual>
+            <geometry>
+                <cylinder length="0.037" radius=".04" />
+            </geometry>
+            <material name="gray" />
+            <origin rpy="1.5708 0 0" xyz="0 0 0" />
+        </visual>
+        <collision>
+            <geometry>
+                <cylinder length="0.037" radius=".04" />
+            </geometry>
+            <material name="gray" />
+            <origin rpy="1.5708 0 0" xyz="0 0 0" />
+        </collision>
+    </link>
+     <link name="wheel4">
+        <xacro:default_inertial mass="1.0"/>
+        <visual>
+            <geometry>
+                <cylinder length="0.037" radius=".04" />
+            </geometry>
+            <material name="gray" />
+            <origin rpy="1.5708 0 0" xyz="0 0 0" />
+        </visual>
+        <collision>
+            <geometry>
+                <cylinder length="0.037" radius=".04" />
+            </geometry>
+            <material name="gray" />
+            <origin rpy="1.5708 0 0" xyz="0 0 0" />
+        </collision>
+    </link>
+        <link name="base_link_r">
+            <xacro:default_inertial mass="0.075"/>
+        <visual>
+            <origin rpy="0 4.7 0" xyz="0.045 0 0"/>
+            <geometry>
+                <mesh filename="package://robertbot_description/mesh/u_type_robot_waist_bracketr.stl" scale="${scaling}"/>
+            </geometry>
+            <material name="brown" />
+        </visual>
+        <collision>
+            <origin rpy="0 4.7 0" xyz="0.045 0 0"/>
+            <geometry>
+                <mesh filename="package://robertbot_description/mesh/u_type_robot_waist_bracketr.stl" scale="${scaling}"/>
+            </geometry>
+        </collision>
+    </link>
+    <link name="base_link_l">
+        <xacro:default_inertial mass="0.075"/>
+        <visual>
+            <origin rpy="0 -4.7 3.14" xyz="0.045 0 0"/>
+            <geometry>
+                <mesh filename="package://robertbot_description/mesh/u_type_robot_waist_bracketl.stl" scale="${scaling}"/>
+            </geometry>
+            <material name="brown" />
+        </visual>
+        <collision>
+            <origin rpy="0 -4.7 3.14" xyz="0.045 0 0"/>
+            <geometry>
+                <mesh filename="package://robertbot_description/mesh/u_type_robot_waist_bracketl.stl" scale="${scaling}"/>
+            </geometry>
+        </collision>
+    </link>
+    <link name="servo1_bracket">
+        <xacro:default_inertial mass="0.025"/>
+        <visual>
+            <origin rpy="1.57 0 0" xyz="-0.01 0.03 0"/>
+            <geometry>
+                <mesh filename="package://robertbot_description/mesh/multi_functional_servo_bracket.stl" scale="${scaling}"/>
+            </geometry>
+            <material name="coolgrey" />
+        </visual>
+        <collision>
+            <origin rpy="1.57 0 0" xyz="-0.01 0.03 0"/>
+            <geometry>
+                <mesh filename="package://robertbot_description/mesh/multi_functional_servo_bracket.stl" scale="${scaling}"/>
+            </geometry>
+            <material name="coolgrey" />
+        </collision>
+    </link>
+    <link name="servo1">
+        <xacro:default_inertial mass="0.05"/>
+        <visual>
+            <origin rpy="0 0 0" xyz="0 0 0"/>
+            <geometry>
+                <mesh filename="package://robertbot_description/mesh/mg996r_servo.stl" scale="${scaling}"/>
+            </geometry>
+            <material name="coolgrey" />
+        </visual>
+        <collision>
+            <origin rpy="0 0 0" xyz="0 0 0"/>
+            <geometry>
+                <mesh filename="package://robertbot_description/mesh/mg996r_servo.stl" scale="${scaling}"/>
+            </geometry>
+            <material name="coolgrey" />
+        </collision>
+    </link>
+    <link name="servo1_horn">
+        <xacro:default_inertial mass="0.005"/>
+        <visual>
+            <origin rpy="1.57 0 0" xyz="0 0 0"/>
+            <geometry>
+                <mesh filename="package://robertbot_description/mesh/aluminum_servo_horn.stl" scale="${scaling}"/>
+            </geometry>
+            <material name="coolgrey" />
+        </visual>
+        <collision>
+            <origin rpy="1.57 0 0" xyz="0 0 0"/>
+            <geometry>
+                <mesh filename="package://robertbot_description/mesh/aluminum_servo_horn.stl" scale="${scaling}"/>
+            </geometry>
+            <material name="coolgrey" />
+        </collision>
+    </link>
+    <link name="servo2_bracket">
+        <xacro:default_inertial mass="0.025"/>
+        <visual>
+            <origin rpy="1.57 1.57 3.14" xyz="0.023 -0.04 0.024"/>
+            <geometry>
+                <mesh filename="package://robertbot_description/mesh/multi_functional_servo_bracket.stl" scale="${scaling}"/>
+            </geometry>
+            <material name="coolgrey" />
+        </visual>
+        <collision>
+            <origin rpy="1.57 1.57 3.14" xyz="0.023 -0.04 0.024"/>
+            <geometry>
+                <mesh filename="package://robertbot_description/mesh/multi_functional_servo_bracket.stl" scale="${scaling}"/>
+            </geometry>
+            <material name="coolgrey" />
+        </collision>
+    </link>
+    <link name="doublelongu_servobracketl">
+        <xacro:default_inertial mass="0.025"/>
+        <visual>
+            <origin rpy="3.14 0 0" xyz="-0.028 0.052 0.015"/>
+            <geometry>
+                <mesh filename="package://robertbot_description/mesh/long_u_type_servo_bracket.stl" scale="${scaling}"/>
+            </geometry>
+            <material name="coolgrey" />
+        </visual>
+        <collision>
+            <origin rpy="3.14 0 0" xyz="-0.028 0.052 0.015"/>
+            <geometry>
+                <mesh filename="package://robertbot_description/mesh/long_u_type_servo_bracket.stl" scale="${scaling}"/>
+            </geometry>
+            <material name="coolgrey" />
+        </collision>
+    </link>
+    <link name="doublelongu_servobracketr">
+        <xacro:default_inertial mass="0.025"/>
+        <visual>
+            <origin rpy="0 0 0" xyz="-0.028 -0.002 -0.01"/>
+            <geometry>
+                <mesh filename="package://robertbot_description/mesh/long_u_type_servo_bracket.stl" scale="${scaling}"/>
+            </geometry>
+            <material name="coolgrey" />
+        </visual>
+        <collision>
+            <origin rpy="0 0 0" xyz="-0.028 -0.002 -0.01"/>
+            <geometry>
+                <mesh filename="package://robertbot_description/mesh/long_u_type_servo_bracket.stl" scale="${scaling}"/>
+            </geometry>
+            <material name="coolgrey" />
+        </collision>
+    </link>
+    <link name="servo2">
+        <xacro:default_inertial mass="0.05"/>
+        <visual>
+            <origin rpy="0 -1.57 0" xyz="0.017 0.001 0.006"/>
+            <geometry>
+                <mesh filename="package://robertbot_description/mesh/mg996r_servo.stl" scale="${scaling}"/>
+            </geometry>
+            <material name="coolgrey" />
+        </visual>
+        <collision>
+            <origin rpy="0 -1.57 0" xyz="0.017 0.001 0.006"/>
+            <geometry>
+                <mesh filename="package://robertbot_description/mesh/mg996r_servo.stl" scale="${scaling}"/>
+            </geometry>
+            <material name="coolgrey" />
+        </collision>
+    </link>
+    <link name="servo2_horn">
+        <xacro:default_inertial mass="0.005"/>
+        <visual>
+            <origin rpy="1.57 1.57 3.14" xyz="-0.001 0.012 -0.002"/>
+            <geometry>
+                <mesh filename="package://robertbot_description/mesh/aluminum_servo_horn.stl" scale="${scaling}"/>
+            </geometry>
+            <material name="coolgrey" />
+        </visual>
+        <collision>
+            <origin rpy="1.57 1.57 3.14" xyz="-0.001 0.012 -0.002"/>
+            <geometry>
+                <mesh filename="package://robertbot_description/mesh/aluminum_servo_horn.stl" scale="${scaling}"/>
+            </geometry>
+            <material name="coolgrey" />
+        </collision>
+    </link>
+    <link name="core_u">
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